File: Plate/Plate.kicad_pcb (KiCad board)
At the start: 2 copper layers, 142.5 x 106.3 mm, 34 parts, among them J1 HOLE, J10 HOLE, J11 HOLE, J12 HOLE, J13 HOLE, J14 HOLE, J15 HOLE, J16 HOLE, J17 HOLE, J18 HOLE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

Commit message: Renamed project
Renamed project to Koca58 because it's now quite different to the
Lily58. Also added fields to parts within KiCad so the python BOM
generator could be removed.
Parts:
- J30, J31, J32, J33, J34: footprint yuchi:M2_HOLE_PCB -> MountingHole:MountingHole_2.2mm_M2_Pad
Other:
- outline, holes or cut-outs redrawn
