File: Plate/Plate.kicad_sch (KiCad schematic)
At the start: 34 parts, among them J1 HOLE, J10 HOLE, J11 HOLE, J12 HOLE, J13 HOLE, J14 HOLE, J15 HOLE, J16 HOLE, J17 HOLE, J18 HOLE, J19 HOLE, J2 HOLE, J20 HOLE, J21 HOLE, J22 HOLE, J23 HOLE, J24 HOLE, J25 HOLE, J26 HOLE, J27 HOLE, J28 HOLE, J29 HOLE, J3 HOLE, J30 M2, J31 M2, J32 M2, J33 M2, J34 M2, J4 HOLE, J5 HOLE, J6 HOLE, J7 HOLE, J8 HOLE, J9 HOLE

Commit message: Renamed project
Renamed project to Koca58 because it's now quite different to the
Lily58. Also added fields to parts within KiCad so the python BOM
generator could be removed.
Parts:
- J30, J31, J32, J33, J34: footprint yuchi:M2_HOLE_PCB -> MountingHole:MountingHole_2.2mm_M2_Pad
Other:
- title: Lily58 Koca Plate -> Koca58 Plate
Changed lines of the file:
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@@
 (kicad_sch
-	(version 20231120)
+	(version 20250114)
 	(generator "eeschema")
-	(generator_version "8.0")
+	(generator_version "9.0")
 	(paper "A4")
 	(title_block
-		(title "Lily58 Koca Plate")
-		(date "2025-01-10")
-		(rev "1")
+		(title "Koca58 Plate")
+		(date "2025-05-10")
+		(rev "v1.0.0")
 	)
 	(no_connect
@@
 			)
 		)
-		(property "Footprint" "yuchi:M2_HOLE_PCB"
+		(property "Footprint" "MountingHole:MountingHole_2.2mm_M2_Pad"
 			(at 106.68 140.97 0)
 			(effects
@@
 			)
 		)
-		(property "Footprint" "yuchi:M2_HOLE_PCB"
+		(property "Footprint" "MountingHole:MountingHole_2.2mm_M2_Pad"
 			(at 119.38 140.97 0)
 			(effects
@@
 			)
 		)
-		(property "Footprint" "yuchi:M2_HOLE_PCB"
+		(property "Footprint" "MountingHole:MountingHole_2.2mm_M2_Pad"
 			(at 93.98 140.97 0)
 			(effects
@@
 			)
 		)
-		(property "Footprint" "yuchi:M2_HOLE_PCB"
+		(property "Footprint" "MountingHole:MountingHole_2.2mm_M2_Pad"
 			(at 81.28 140.97 0)
 			(effects
@@
 			)
 		)
-		(property "Footprint" "yuchi:M2_HOLE_PCB"
+		(property "Footprint" "MountingHole:MountingHole_2.2mm_M2_Pad"
 			(at 130.81 140.97 0)
 			(effects
@@
 		)
 	)
+	(embedded_fonts no)
 )
