File: PCB/Koca58.kicad_sch (KiCad schematic)
At the start: 166 parts, among them J1 USB_C_Receptacle_USB2.0_16P, J2 Conn_01x04_Pin, J3 Conn_01x04_Pin, J4 RJ45, J5 USB_C_Receptacle_USB2.0_16P, J6 Conn_01x04_Pin, J7 Conn_01x04_Pin, J8 RJ45, SW1 SW_Push, SW10 MX_SWITCH, SW11 MX_SWITCH, SW12 MX_SWITCH, SW13 MX_SWITCH, SW14 MX_SWITCH, SW15 MX_SWITCH, SW16 MX_SWITCH, SW17 MX_SWITCH, SW18 MX_SWITCH, SW19 MX_SWITCH, SW2 MX_SWITCH, SW20 MX_SWITCH, SW21 MX_SWITCH, SW22 MX_SWITCH, SW23 MX_SWITCH, SW24 MX_SWITCH, SW25 MX_SWITCH, SW26 MX_SWITCH, SW27 MX_SWITCH, SW28 MX_SWITCH, SW29 MX_SWITCH, SW3 MX_SWITCH, SW30 MX_SWITCH, SW31 MX_SWITCH, SW32 MX_SWITCH, SW33 MX_SWITCH, SW34 MX_SWITCH, SW35 MX_SWITCH, SW36 MX_SWITCH, SW37 SW_Push, SW38 MX_SWITCH, SW39 MX_SWITCH, SW4 MX_SWITCH, SW40 MX_SWITCH, SW41 MX_SWITCH, SW42 MX_SWITCH, SW43 MX_SWITCH, SW44 MX_SWITCH, SW45 MX_SWITCH, SW46 MX_SWITCH, SW47 MX_SWITCH, SW48 MX_SWITCH, SW49 MX_SWITCH, SW5 MX_SWITCH, SW50 MX_SWITCH, SW51 MX_SWITCH, SW52 MX_SWITCH, SW53 MX_SWITCH, SW54 MX_SWITCH, SW55 MX_SWITCH, SW56 MX_SWITCH, SW57 MX_SWITCH, SW58 MX_SWITCH, SW59 MX_SWITCH, SW6 MX_SWITCH, SW60 MX_SWITCH, SW7 MX_SWITCH, SW8 MX_SWITCH, SW9 MX_SWITCH, U1 USBLC6-2SC6, U2 STM32F103RCTx, U3 USBLC6-2SC6, U4 AMS1117-3.3, U5 USBLC6-2SC6, U6 STM32F103RCTx, U7 USBLC6-2SC6, U8 AMS1117-3.3, Y1 12Mhz, Y2 12Mhz

Commit message: Added new case files
Also did some minor changes to the main PCB
Parts:
- U2, U6: LCSC/JLC Part Number C39704 -> C8323; Manufacturer Part Number STM32F103RCT6TR -> STM32F103RCT6
Connections:
- net CON_RX_L: now also R9.1; no longer R7.1
- net CON_TX_L: now also R7.1; no longer R9.1
- net RX_L: now also U3.3 (I/O2); no longer U3.1 (I/O1)
- net TX_L: now also U3.1 (I/O1); no longer U3.3 (I/O2)
Other:
- note added: "Power Flags"

Commit message: Improved via to pad spacing
Fab complained
Parts:
- SW1, SW37: footprint Button_Switch_SMD:SW_SPST_CK_RS282G05A3 -> Koca58:Korean Hroparts Elec K2-1107ST-A4DW-06
Changed lines of the file:
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@@
 	(title_block
 		(title "Koca58")
-		(date "2025-05-18")
-		(rev "v1.0.1")
+		(date "2025-05-27")
+		(rev "v1.0.2")
 		(company "oxnh")
 	)
@@
 			)
 		)
-		(property "Footprint" "Button_Switch_SMD:SW_SPST_CK_RS282G05A3"
+		(property "Footprint" "Koca58:Korean Hroparts Elec K2-1107ST-A4DW-06"
 			(at 369.57 261.62 0)
 			(show_name yes)
@@
 			)
 		)
-		(property "Footprint" "Button_Switch_SMD:SW_SPST_CK_RS282G05A3"
+		(property "Footprint" "Koca58:Korean Hroparts Elec K2-1107ST-A4DW-06"
 			(at 369.57 62.23 0)
 			(show_name yes)
