File: PCB/Koca58.kicad_sch (KiCad schematic)
At the start: 166 parts, among them J1 USB_C_Receptacle_USB2.0_16P, J2 Conn_01x04_Pin, J3 Conn_01x04_Pin, J4 RJ45, J5 USB_C_Receptacle_USB2.0_16P, J6 Conn_01x04_Pin, J7 Conn_01x04_Pin, J8 RJ45, SW1 SW_Push, SW10 MX_SWITCH, SW11 MX_SWITCH, SW12 MX_SWITCH, SW13 MX_SWITCH, SW14 MX_SWITCH, SW15 MX_SWITCH, SW16 MX_SWITCH, SW17 MX_SWITCH, SW18 MX_SWITCH, SW19 MX_SWITCH, SW2 MX_SWITCH, SW20 MX_SWITCH, SW21 MX_SWITCH, SW22 MX_SWITCH, SW23 MX_SWITCH, SW24 MX_SWITCH, SW25 MX_SWITCH, SW26 MX_SWITCH, SW27 MX_SWITCH, SW28 MX_SWITCH, SW29 MX_SWITCH, SW3 MX_SWITCH, SW30 MX_SWITCH, SW31 MX_SWITCH, SW32 MX_SWITCH, SW33 MX_SWITCH, SW34 MX_SWITCH, SW35 MX_SWITCH, SW36 MX_SWITCH, SW37 SW_Push, SW38 MX_SWITCH, SW39 MX_SWITCH, SW4 MX_SWITCH, SW40 MX_SWITCH, SW41 MX_SWITCH, SW42 MX_SWITCH, SW43 MX_SWITCH, SW44 MX_SWITCH, SW45 MX_SWITCH, SW46 MX_SWITCH, SW47 MX_SWITCH, SW48 MX_SWITCH, SW49 MX_SWITCH, SW5 MX_SWITCH, SW50 MX_SWITCH, SW51 MX_SWITCH, SW52 MX_SWITCH, SW53 MX_SWITCH, SW54 MX_SWITCH, SW55 MX_SWITCH, SW56 MX_SWITCH, SW57 MX_SWITCH, SW58 MX_SWITCH, SW59 MX_SWITCH, SW6 MX_SWITCH, SW60 MX_SWITCH, SW7 MX_SWITCH, SW8 MX_SWITCH, SW9 MX_SWITCH, U1 USBLC6-2SC6, U2 STM32F103RCTx, U3 USBLC6-2SC6, U4 AMS1117-3.3, U5 USBLC6-2SC6, U6 STM32F103RCTx, U7 USBLC6-2SC6, U8 AMS1117-3.3, Y1 12Mhz, Y2 12Mhz

Commit message: Re-routed PCB
Both keyboard sides were completely rerouted so
that all components are on the top-side (except for hotswap sockets).

Also reduced BOM slightly and switched to a better linear regulator.
This change also reduced the total VBUS capacitance to under 10uF,
making the device properly meet the USB-C spec.

USB-C differential pairs also have 90 ohm differential impedance now,
and have matched lengths. Trace width and gap was calculated using
JLCPCB controlled impedance calculator.
Parts:
- removed C3: 1u, Capacitor_SMD:C_0402_1005Metric, symbol Device:C
- removed C4: 10u, Capacitor_SMD:C_0603_1608Metric, symbol Device:C
- removed F1, F2: Polyfuse, Fuse:Fuse_0603_1608Metric, symbol Device:Polyfuse
- removed FB1, FB2: 120R, Resistor_SMD:R_0603_1608Metric, symbol Device:FerriteBead
- removed JP1, JP3: SolderJumper_2_Open, Jumper:SolderJumper-2_P1.3mm_Open_Pad1.0x1.5mm, symbol Jumper:SolderJumper_2_Open
- removed R14, R4: 10k, Resistor_SMD:R_0402_1005Metric, symbol Device:R
- removed TP1, TP2: TestPoint, TestPoint:TestPoint_Pad_D1.0mm, symbol Connector:TestPoint
- removed U4, U8: AMS1117-3.3, Package_TO_SOT_SMD:SOT-89-3, symbol Regulator_Linear:AMS1117-3.3
- added C28, C29: 100n, Capacitor_SMD:C_0402_1005Metric, symbol Device:C
- added U10, U9: AP2112K-3.3, Package_TO_SOT_SMD:SOT-23-5, symbol Regulator_Linear:AP2112K-3.3
- C12, C13, C25, C26: value 22u -> 4.7u; LCSC/JLC Part Number C59461 -> C19666; Manufacturer Part Number CL10A226MQ8NRNC -> CL10A475KO8NNNC
- C16: value 1u -> 4.7u; footprint Capacitor_SMD:C_0402_1005Metric -> Capacitor_SMD:C_0603_1608Metric; LCSC/JLC Part Number C52923 -> C19666; Manufacturer Part Number CL05A105KA5NQNC -> CL10A475KO8NNNC
- C17: value 10u -> 4.7u; LCSC/JLC Part Number C96446 -> C19666; Manufacturer Part Number CL10A106MA8NRNC -> CL10A475KO8NNNC
- J2, J6: footprint Koca58:SWD_POGO -> Koca58:SWD_POGO_P1.27
Connections:
- net JMP_BOOT0_L is gone; now on net B0_L: R5.2
- net JMP_BOOT0_R is gone; now on net B0_R: R15.2
- net VBUS is gone; now on net VBUS_R: J5.A4 (VBUS), J5.A9 (VBUS), J5.B4 (VBUS), J5.B9 (VBUS), R18.2, U5.5 (VBUS), U7.5 (VBUS)
- net VDC is gone; now on net VBUS_L: J1.A4 (VBUS), J1.A9 (VBUS), J1.B4 (VBUS), J1.B9 (VBUS), R8.2, U1.5 (VBUS), U3.5 (VBUS)
- net VDDA_L is gone; now on net +3V3_L: C1.1, C2.1, U2.13 (VDDA)
- net VDDA_R is gone; now on net +3V3_R: C14.1, C15.1, U6.13 (VDDA)
- net NRST_L: now also C28.1
- net NRST_R: now also C29.1
- net +3.3VA renamed +3V3_R
- net +3V3_R: now also U10.5 (VOUT); no longer C16.1
- net +3V3 renamed +3V3_L
- net +3V3_L: now also C16.1, U9.5 (VOUT)
- net +5V renamed VBUS_L
- net VBUS_L: now also U9.1 (VIN), U9.3 (EN)
- net +5VA renamed VBUS_R
- net VBUS_R: now also U10.1 (VIN), U10.3 (EN)
- net GND renamed GND_L
- net GND_L: now also C16.2, C28.2, U9.2 (GND)
- net GNDA renamed GND_R
- net GND_R: now also C29.2, U10.2 (GND); no longer C16.2
- net TP_L: no longer names the net of U2.61 (PB8)
- net TP_R: no longer names the net of U6.61 (PB8)
- no-connect marks 50 -> 52
Other:
- note removed: "Boot jumper"
- note removed: "SW Debug"
- note removed: "VDDA filtering"
- moved on the sheet: C1, C14, C15, C2, R15, R5, SW1, SW37
