File: PCB/Koca58.kicad_pcb (KiCad board)
At the start: 2 copper layers, 290.1 x 131 mm, 166 parts, among them J1 USB_C_Receptacle_USB2.0_16P, J2 Conn_01x04_Pin, J3 Conn_01x04_Pin, J4 RJ45, J5 USB_C_Receptacle_USB2.0_16P, J6 Conn_01x04_Pin, J7 Conn_01x04_Pin, J8 RJ45, SW1 SW_Push, SW10 MX_SWITCH, SW11 MX_SWITCH, SW12 MX_SWITCH, SW13 MX_SWITCH, SW14 MX_SWITCH, SW15 MX_SWITCH, SW16 MX_SWITCH, SW17 MX_SWITCH, SW18 MX_SWITCH, SW19 MX_SWITCH, SW2 MX_SWITCH, SW20 MX_SWITCH, SW21 MX_SWITCH, SW22 MX_SWITCH, SW23 MX_SWITCH, SW24 MX_SWITCH, SW25 MX_SWITCH, SW26 MX_SWITCH, SW27 MX_SWITCH, SW28 MX_SWITCH, SW29 MX_SWITCH, SW3 MX_SWITCH, SW30 MX_SWITCH, SW31 MX_SWITCH, SW32 MX_SWITCH, SW33 MX_SWITCH, SW34 MX_SWITCH, SW35 MX_SWITCH, SW36 MX_SWITCH, SW37 SW_Push, SW38 MX_SWITCH, SW39 MX_SWITCH, SW4 MX_SWITCH, SW40 MX_SWITCH, SW41 MX_SWITCH, SW42 MX_SWITCH, SW43 MX_SWITCH, SW44 MX_SWITCH, SW45 MX_SWITCH, SW46 MX_SWITCH, SW47 MX_SWITCH, SW48 MX_SWITCH, SW49 MX_SWITCH, SW5 MX_SWITCH, SW50 MX_SWITCH, SW51 MX_SWITCH, SW52 MX_SWITCH, SW53 MX_SWITCH, SW54 MX_SWITCH, SW55 MX_SWITCH, SW56 MX_SWITCH, SW57 MX_SWITCH, SW58 MX_SWITCH, SW59 MX_SWITCH, SW6 MX_SWITCH, SW60 MX_SWITCH, SW7 MX_SWITCH, SW8 MX_SWITCH, SW9 MX_SWITCH, U1 USBLC6-2SC6, U2 STM32F103RCTx, U3 USBLC6-2SC6, U4 AMS1117-3.3, U5 USBLC6-2SC6, U6 STM32F103RCTx, U7 USBLC6-2SC6, U8 AMS1117-3.3, Y1 12Mhz, Y2 12Mhz

Commit message: Re-routed PCB
Both keyboard sides were completely rerouted so
that all components are on the top-side (except for hotswap sockets).

Also reduced BOM slightly and switched to a better linear regulator.
This change also reduced the total VBUS capacitance to under 10uF,
making the device properly meet the USB-C spec.

USB-C differential pairs also have 90 ohm differential impedance now,
and have matched lengths. Trace width and gap was calculated using
JLCPCB controlled impedance calculator.
Parts:
- removed C3: 1u, Capacitor_SMD:C_0402_1005Metric
- removed C4: 10u, Capacitor_SMD:C_0603_1608Metric
- removed F1, F2: Polyfuse, Fuse:Fuse_0603_1608Metric
- removed FB1, FB2: 120R, Resistor_SMD:R_0603_1608Metric
- removed JP1, JP3: SolderJumper_2_Open, Jumper:SolderJumper-2_P1.3mm_Open_Pad1.0x1.5mm
- removed R14, R4: 10k, Resistor_SMD:R_0402_1005Metric
- removed TP1, TP2: TestPoint, TestPoint:TestPoint_Pad_D1.0mm
- removed U4, U8: AMS1117-3.3, Package_TO_SOT_SMD:SOT-89-3
- added C28: 100n, Capacitor_SMD:C_0402_1005Metric, F.Cu at (186.3, 124.0)
- added C29: 100n, Capacitor_SMD:C_0402_1005Metric, F.Cu at (222.0, 124.1)
- added U10: AP2112K-3.3, Package_TO_SOT_SMD:SOT-23-5, F.Cu at (233.8, 106.6)
- added U9: AP2112K-3.3, Package_TO_SOT_SMD:SOT-23-5, F.Cu at (174.3, 106.8)
- C12, C13, C25, C26: value 22u -> 4.7u; moved to F.Cu
- C16: value 1u -> 4.7u; footprint Capacitor_SMD:C_0402_1005Metric -> Capacitor_SMD:C_0603_1608Metric
- C17: value 10u -> 4.7u
- J2, J6: footprint Koca58:SWD_POGO -> Koca58:SWD_POGO_P1.27; moved to F.Cu
- R1, R11, R12, R2: moved to F.Cu
- moved C16 49.5 mm to (178.0, 120.8), turned to 90 degrees
- moved C25 23.6 mm to (234.3, 103.8)
- moved C26 23.5 mm to (233.9, 109.5)
- moved C12 21.6 mm to (174.8, 103.9)
- moved C13 21.1 mm to (174.3, 109.7)
- moved C17 13.4 mm to (213.7, 120.8), turned to 90 degrees
- moved J2 11.0 mm to (180.1, 111.3), turned to 45 degrees
- moved J6 7.57 mm to (215.1, 111.0), turned to 45 degrees
- moved R11 5.96 mm to (234.9, 96.0), turned to 180 degrees
- moved R1 4.75 mm to (182.9, 103.3), turned to 90 degrees
- moved C11 4.63 mm to (186.4, 126.2)
- moved Y1 4.47 mm to (184.8, 128.4)
- moved C10 4.31 mm to (183.9, 126.2)
- moved C9 4.05 mm to (182.2, 124.0)
- moved R5 4.04 mm to (177.1, 118.6)
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Connections:
- C1 pad 1: /VDDA_L -> +3V3_L
- C1 pad 2: GND -> GND_L
- C10 pad 2: GND -> GND_L
- C11 pad 2: GND -> GND_L
- C12 pad 1: +5V -> VBUS_L
- C12 pad 2: GND -> GND_L
- C13 pad 1: +3V3 -> +3V3_L
- C13 pad 2: GND -> GND_L
- C14 pad 1: /VDDA_R -> +3V3_R
- C14 pad 2: GNDA -> GND_R
- C15 pad 1: /VDDA_R -> +3V3_R
- C15 pad 2: GNDA -> GND_R
- C16 pad 1: +3.3VA -> +3V3_L
- C16 pad 2: GNDA -> GND_L
- C17 pad 1: +3.3VA -> +3V3_R
- C17 pad 2: GNDA -> GND_R
- C18 pad 1: +3.3VA -> +3V3_R
- C18 pad 2: GNDA -> GND_R
- C19 pad 1: +3.3VA -> +3V3_R
- C19 pad 2: GNDA -> GND_R
- C2 pad 1: /VDDA_L -> +3V3_L
- C2 pad 2: GND -> GND_L
- C20 pad 1: +3.3VA -> +3V3_R
- C20 pad 2: GNDA -> GND_R
- C21 pad 1: +3.3VA -> +3V3_R
- C21 pad 2: GNDA -> GND_R
- C22 pad 1: +3.3VA -> +3V3_R
- C22 pad 2: GNDA -> GND_R
- C23 pad 2: GNDA -> GND_R
- C24 pad 2: GNDA -> GND_R
- C25 pad 1: +5VA -> VBUS_R
- C25 pad 2: GNDA -> GND_R
- C26 pad 1: +3.3VA -> +3V3_R
- C26 pad 2: GNDA -> GND_R
- C5 pad 1: +3V3 -> +3V3_L
- C5 pad 2: GND -> GND_L
- C6 pad 1: +3V3 -> +3V3_L
- C6 pad 2: GND -> GND_L
- C7 pad 1: +3V3 -> +3V3_L
- C7 pad 2: GND -> GND_L
- C8 pad 1: +3V3 -> +3V3_L
- C8 pad 2: GND -> GND_L
- C9 pad 1: +3V3 -> +3V3_L
- C9 pad 2: GND -> GND_L
- J1 pad A1: GND -> GND_L
- J1 pad A12: GND -> GND_L
- J1 pad A4: VDC -> VBUS_L
- J1 pad A9: VDC -> VBUS_L
- J1 pad B1: GND -> GND_L
- J1 pad B12: GND -> GND_L
- J1 pad B4: VDC -> VBUS_L
- J1 pad B9: VDC -> VBUS_L
- J1 pad S1: GND -> GND_L
- J2 pad 1: GND -> GND_L
- J2 pad 4: +3V3 -> +3V3_L
- J3 pad 1: GND -> GND_L
- J3 pad 2: +3V3 -> +3V3_L
- J4 pad 7: GND -> GND_L
- J4 pad 8: GND -> GND_L
- J5 pad A1: GNDA -> GND_R
- J5 pad A12: GNDA -> GND_R
- J5 pad A4: VBUS -> VBUS_R
- J5 pad A9: VBUS -> VBUS_R
- J5 pad B1: GNDA -> GND_R
- J5 pad B12: GNDA -> GND_R
- J5 pad B4: VBUS -> VBUS_R
- J5 pad B9: VBUS -> VBUS_R
- J5 pad S1: GNDA -> GND_R
- J6 pad 1: GNDA -> GND_R
- J6 pad 4: +3.3VA -> +3V3_R
- J7 pad 1: GNDA -> GND_R
- J7 pad 2: +3.3VA -> +3V3_R
- J8 pad 7: GNDA -> GND_R
- J8 pad 8: GNDA -> GND_R
- JP2 pad 1: +3V3 -> +3V3_L
- JP4 pad 1: +3.3VA -> +3V3_R
- R1 pad 1: GND -> GND_L
- R10 pad 2: GND -> GND_L
- R11 pad 1: GNDA -> GND_R
- R12 pad 1: GNDA -> GND_R
- R13 pad 1: +3.3VA -> +3V3_R
- R15 pad 1: GNDA -> GND_R
- R15 pad 2: /JMP_BOOT0_R -> /B0_R
- R16 pad 2: GNDA -> GND_R
- R18 pad 2: VBUS -> VBUS_R
- R2 pad 1: GND -> GND_L
- R20 pad 2: GNDA -> GND_R
- R3 pad 1: +3V3 -> +3V3_L
- R5 pad 1: GND -> GND_L
- R5 pad 2: /JMP_BOOT0_L -> /B0_L
- R6 pad 2: +3V3 -> +3V3_L
- R8 pad 2: VDC -> VBUS_L
- SW1 pad 1: GND -> GND_L
- SW10 pad 1: GND -> GND_L
- SW11 pad 1: GND -> GND_L
- SW12 pad 1: GND -> GND_L
- SW13 pad 1: GND -> GND_L
- SW14 pad 1: GND -> GND_L
- SW15 pad 1: GND -> GND_L
- SW16 pad 1: GND -> GND_L
- SW17 pad 1: GND -> GND_L
- SW18 pad 1: GND -> GND_L
- SW19 pad 1: GND -> GND_L
- SW2 pad 1: GND -> GND_L
- SW20 pad 1: GND -> GND_L
- SW21 pad 1: GND -> GND_L
- SW22 pad 1: GND -> GND_L
- SW23 pad 1: GND -> GND_L
- SW24 pad 1: GND -> GND_L
- SW25 pad 1: GND -> GND_L
- SW26 pad 1: GND -> GND_L
- SW27 pad 1: GND -> GND_L
- SW28 pad 1: GND -> GND_L
- SW29 pad 1: GND -> GND_L
- SW3 pad 1: GND -> GND_L
- SW30 pad 1: GND -> GND_L
- SW31 pad 1: GNDA -> GND_R
- SW32 pad 1: GNDA -> GND_R
- SW33 pad 1: GNDA -> GND_R
- SW34 pad 1: GNDA -> GND_R
- SW35 pad 1: GNDA -> GND_R
- SW36 pad 1: GNDA -> GND_R
- SW37 pad 1: GNDA -> GND_R
- SW38 pad 1: GNDA -> GND_R
- SW39 pad 1: GNDA -> GND_R
- SW4 pad 1: GND -> GND_L
- SW40 pad 1: GNDA -> GND_R
- SW41 pad 1: GNDA -> GND_R
- SW42 pad 1: GNDA -> GND_R
- SW43 pad 1: GNDA -> GND_R
- SW44 pad 1: GNDA -> GND_R
- SW45 pad 1: GNDA -> GND_R
- SW46 pad 1: GNDA -> GND_R
- SW47 pad 1: GNDA -> GND_R
- SW48 pad 1: GNDA -> GND_R
- SW49 pad 1: GNDA -> GND_R
- SW5 pad 1: GND -> GND_L
- SW50 pad 1: GNDA -> GND_R
- SW51 pad 1: GNDA -> GND_R
- SW52 pad 1: GNDA -> GND_R
- SW53 pad 1: GNDA -> GND_R
- SW54 pad 1: GNDA -> GND_R
- SW55 pad 1: GNDA -> GND_R
- SW56 pad 1: GNDA -> GND_R
- SW57 pad 1: GNDA -> GND_R
- SW58 pad 1: GNDA -> GND_R
- SW59 pad 1: GNDA -> GND_R
- SW6 pad 1: GND -> GND_L
- SW60 pad 1: GNDA -> GND_R
- SW7 pad 1: GND -> GND_L
- SW8 pad 1: GND -> GND_L
- SW9 pad 1: GND -> GND_L
- U1 pad 2: GND -> GND_L
- U1 pad 5: VDC -> VBUS_L
- U2 pad 1: +3V3 -> +3V3_L
- U2 pad 12: GND -> GND_L
- U2 pad 13: /VDDA_L -> +3V3_L
- U2 pad 18: GND -> GND_L
- U2 pad 19: +3V3 -> +3V3_L
- U2 pad 31: GND -> GND_L
- U2 pad 32: +3V3 -> +3V3_L
- U2 pad 47: GND -> GND_L
- U2 pad 48: +3V3 -> +3V3_L
- U2 pad 61: TP_L -> unconnected-(U2-PB8-Pad61)
- U2 pad 63: GND -> GND_L
- U2 pad 64: +3V3 -> +3V3_L
- U3 pad 2: GND -> GND_L
- U3 pad 5: VDC -> VBUS_L
- U5 pad 2: GNDA -> GND_R
- U5 pad 5: VBUS -> VBUS_R
- U6 pad 1: +3.3VA -> +3V3_R
- U6 pad 12: GNDA -> GND_R
- U6 pad 13: /VDDA_R -> +3V3_R
- U6 pad 18: GNDA -> GND_R
- U6 pad 19: +3.3VA -> +3V3_R
- U6 pad 31: GNDA -> GND_R
- U6 pad 32: +3.3VA -> +3V3_R
- U6 pad 47: GNDA -> GND_R
- U6 pad 48: +3.3VA -> +3V3_R
- U6 pad 61: TP_R -> unconnected-(U6-PB8-Pad61)
- U6 pad 63: GNDA -> GND_R
- U6 pad 64: +3.3VA -> +3V3_R
- U7 pad 2: GNDA -> GND_R
- U7 pad 5: VBUS -> VBUS_R
- Y1 pad 2: GND -> GND_L
- Y1 pad 4: GND -> GND_L
- Y2 pad 2: GNDA -> GND_R
- Y2 pad 4: GNDA -> GND_R
Routing:
- net +3V3: track 146.7 -> 0.00 mm, vias 8 -> 0
- net +3.3VA: track 115.4 -> 0.00 mm, vias 9 -> 0
- net +3V3_L: track 0.00 -> 110.2 mm, vias 0 -> 11
- net +3V3_R: track 0.00 -> 100.7 mm, vias 0 -> 8
- net VDC: track 59.3 -> 0.00 mm, vias 3 -> 0
- net VBUS_L: track 0.00 -> 57.5 mm, vias 0 -> 2
- net VBUS: track 53.5 -> 0.00 mm, vias 2 -> 0
- net VBUS_R: track 0.00 -> 51.2 mm
- net L11: track 29.7 -> 78.6 mm
- net GNDA: track 36.3 -> 0.00 mm, vias 78 -> 0
- net GND: track 34.3 -> 0.00 mm, vias 77 -> 0
- net L24: track 137.2 -> 103.7 mm
- net GND_R: track 0.00 -> 31.8 mm, vias 0 -> 23
- net GND_L: track 0.00 -> 31.5 mm, vias 0 -> 22
- net L23: track 94.3 -> 63.5 mm
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- added copper zone on F.Cu, net +3V3_L
- added copper zone on F.Cu, net +3V3_R
- added copper zone on B.Cu, net GND_L
- added copper zone on F.Cu, net GND_L
- added copper zone on B.Cu, net GND_R
- added copper zone on F.Cu, net GND_R
- added copper zone on F.Cu, net VBUS_L
- added copper zone on F.Cu, net VBUS_R
- removed copper zone on B.Cu, net +5V
- removed copper zone on B.Cu, net +5VA
- removed copper zone on B.Cu, net GND
- removed copper zone on F.Cu, net GND
- removed copper zone on B.Cu, net GNDA
- removed copper zone on F.Cu, net GNDA
Other:
- board text added: "Koca58 V1.1.0"
- board text added: "Koca58 v1.1.0"
- board text added: "Koca58 v1.1.0 2026-08-27"
- board text removed: "+ DIO CLK -"
- board text removed: "BOOT0"
- board text removed: "Koca58 V1.0.3"
- board text removed: "Koca58 v1.0.3"
- board text removed: "Koca58 v1.0.3 2025-05-27"
- board text removed: "LEDJPR"
- board text removed: "Yes, I know there are a lot of traces really close together. All of those are for detecting key presses with the direct matrix, so they're really low speed. So I'm not concerned about cross-talk. A direct matrix also seems like an odd choice. Initially I selected it so diodes didn't have to be soldered to the underside of the board. This was intended as a cost saving measure. Howevever, as I iter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"
